File: Neopixel_pico_arcade.kicad_pcb (KiCad board)
At the start: 0 parts

Commit message: Adds basic PCB file with board outline
Other:
- board outline added: 100 x 100 mm
- copper layers 0 -> 4
Changed lines of the file:
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@@
-(kicad_pcb (version 20210228) (generator pcbnew)
+(kicad_pcb (version 20210824) (generator pcbnew)
+  (general
+    (thickness 4.69)
+  )
+  (paper "A4")
+  (layers
+    (0 "F.Cu" signal)
+    (1 "In1.Cu" signal)
+    (2 "In2.Cu" signal)
+    (31 "B.Cu" signal)
+    (32 "B.Adhes" user "B.Adhesive")
+    (33 "F.Adhes" user "F.Adhesive")
+    (34 "B.Paste" user)
+    (35 "F.Paste" user)
+    (36 "B.SilkS" user "B.Silkscreen")
+    (37 "F.SilkS" user "F.Silkscreen")
+    (38 "B.Mask" user)
+    (39 "F.Mask" user)
+    (40 "Dwgs.User" user "User.Drawings")
+    (41 "Cmts.User" user "User.Comments")
+    (42 "Eco1.User" user "User.Eco1")
+    (43 "Eco2.User" user "User.Eco2")
+    (44 "Edge.Cuts" user)
+    (45 "Margin" user)
+    (46 "B.CrtYd" user "B.Courtyard")
+    (47 "F.CrtYd" user "F.Courtyard")
+    (48 "B.Fab" user)
+    (49 "F.Fab" user)
+    (50 "User.1" user)
+    (51 "User.2" user)
+    (52 "User.3" user)
+    (53 "User.4" user)
+    (54 "User.5" user)
+    (55 "User.6" user)
+    (56 "User.7" user)
+    (57 "User.8" user)
+    (58 "User.9" user)
+  )
+  (setup
+    (stackup
+      (layer "F.SilkS" (type "Top Silk Screen"))
+      (layer "F.Paste" (type "Top Solder Paste"))
+      (layer "F.Mask" (type "Top Solder Mask") (color "Green") (thickness 0.01))
+      (layer "F.Cu" (type "copper") (thickness 0.035))
+      (layer "dielectric 1" (type "core") (thickness 1.51) (material "FR4") (epsilon_r 4.5) (loss_tangent 0.02))
+      (layer "In1.Cu" (type "copper") (thickness 0.035))
+      (layer "dielectric 2" (type "prepreg") (thickness 1.51) (material "FR4") (epsilon_r 4.5) (loss_tangent 0.02))
+      (layer "In2.Cu" (type "copper") (thickness 0.035))
+      (layer "dielectric 3" (type "core") (thickness 1.51) (material "FR4") (epsilon_r 4.5) (loss_tangent 0.02))
+      (layer "B.Cu" (type "copper") (thickness 0.035))
+      (layer "B.Mask" (type "Bottom Solder Mask") (color "Green") (thickness 0.01))
+      (layer "B.Paste" (type "Bottom Solder Paste"))
+      (layer "B.SilkS" (type "Bottom Silk Screen"))
+      (copper_finish "None")
+      (dielectric_constraints no)
+    )
+    (pad_to_mask_clearance 0)
+    (pcbplotparams
+      (layerselection 0x00010fc_ffffffff)
+      (disableapertmacros false)
+      (usegerberextensions false)
+      (usegerberattributes true)
+      (usegerberadvancedattributes true)
+      (creategerberjobfile true)
+      (svguseinch false)
+      (svgprecision 6)
+      (excludeedgelayer true)
+      (plotframeref false)
+      (viasonmask false)
+      (mode 1)
+      (useauxorigin false)
+      (hpglpennumber 1)
+      (hpglpenspeed 20)
+      (hpglpendiameter 15.000000)
+      (dxfpolygonmode true)
+      (dxfimperialunits true)
+      (dxfusepcbnewfont true)
+      (psnegative false)
+      (psa4output false)
+      (plotreference true)
+      (plotvalue true)
+      (plotinvisibletext false)
+      (sketchpadsonfab false)
+      (subtractmaskfromsilk false)
+      (outputformat 1)
+      (mirror false)
+      (drillshape 1)
+      (scaleselection 1)
+      (outputdirectory "")
+    )
+  )
+  (net 0 "")
+  (gr_line (start 100 53) (end 100 147) (layer "Edge.Cuts") (width 0.1))
+  (gr_line (start 103 150) (end 197 150) (layer "Edge.Cuts") (width 0.1))
+  (gr_arc (start 103 147) (end 100 147) (angle -90) (layer "Edge.Cuts") (width 0.1))
+  (gr_arc (start 103 53) (end 103 50) (angle -90) (layer "Edge.Cuts") (width 0.1))
+  (gr_arc (start 197 147) (end 197 150) (angle -90) (layer "Edge.Cuts") (width 0.1))
+  (gr_arc (start 197 53) (end 200 53) (angle -90) (layer "Edge.Cuts") (width 0.1))
+  (gr_line (start 200 147) (end 200 53) (layer "Edge.Cuts") (width 0.1))
+  (gr_line (start 103 50) (end 197 50) (layer "Edge.Cuts") (width 0.1))
+  (gr_line (start 110 140) (end 110 60) (layer "F.Fab") (width 0.1))
+  (gr_line (start 110 60) (end 190 60) (layer "F.Fab") (width 0.1))
+  (gr_line (start 190 140) (end 110 140) (layer "F.Fab") (width 0.1))
+  (gr_line (start 190 60) (end 190 140) (layer "F.Fab") (width 0.1))
 )
