File: Neopixel_pico_arcade.kicad_sch (KiCad schematic)
At the start: 19 parts, among them J1 SWD_connector, J2 NES_controller_connector, J3 USB_C_Receptacle_USB2.0, Q1 2N7002, U1 RP2040_Stamp, U2 SN74LV1T34DBV, U3 SRV05-4HTG-D

Commit message: Switches SWD connector to SDM pin headers
Parts:
- J1: footprint Connector_PinHeader_2.54mm:PinHeader_1x03_P2.54mm_Vertical -> Connector_PinHeader_2.54mm:PinHeader_1x03_P2.54mm_Vertical_SMD_Pin1Left
Changed lines of the file:
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@@
     (property "Reference" "J1" (id 0) (at 88.4174 38.8578 0))
     (property "Value" "SWD_connector" (id 1) (at 88.4174 41.1565 0))
-    (property "Footprint" "Connector_PinHeader_2.54mm:PinHeader_1x03_P2.54mm_Vertical" (id 2) (at 81.28 46.99 0)
+    (property "Footprint" "Connector_PinHeader_2.54mm:PinHeader_1x03_P2.54mm_Vertical_SMD_Pin1Left" (id 2) (at 81.28 46.99 0)
       (effects (font (size 1.27 1.27)) hide)
     )
@@
     )
     (path "/2d555828-831d-4418-8791-29126d2f97c5"
-      (reference "J1") (unit 1) (value "SWD_connector") (footprint "Connector_PinHeader_2.54mm:PinHeader_1x03_P2.54mm_Vertical")
+      (reference "J1") (unit 1) (value "SWD_connector") (footprint "Connector_PinHeader_2.54mm:PinHeader_1x03_P2.54mm_Vertical_SMD_Pin1Left")
     )
     (path "/0d864839-2792-4de0-80be-2a96e9fb5773"
